File: physical robot/PCB/Camera/Camera.kicad_sch (KiCad schematic)
At the start: 8 parts, among them U1 ESP32-WROOM-32, U2 OV5640

Commit message: pcb finiished
Parts:
- added C1, C2, C7: 22uF/10V(20%), Capacitor_SMD:C_0603_1608Metric, symbol Device:C
- added C3: 4.7uF/6.3V(10%), Capacitor_SMD:C_0402_1005Metric, symbol Device:C
- added C4, C9: 0.1uF/50V(10%)(NC), Capacitor_SMD:C_0402_1005Metric, symbol Device:C
- added C5, C6, C8: 0.1uF/50V(10%), Capacitor_SMD:C_0402_1005Metric, symbol Device:C
- added D2, D3, D4: LESD5D5.0CT1G, LESD5D5.0CT1G:LESD5D50CT1G, symbol LESD5D5.0CT1G:LESD5D5.0CT1G
- added D4, D6: LED, LED_SMD:LED_0603_1608Metric, symbol Device:LED
- added D5: BAT760-7, BAT760-7:SOD2513X120N, symbol BAT760-7:BAT760-7
- added IC1: AMS1117-3.3, AMS1117-3.3:SOT229P700X180-4N, symbol AMS1117-3.3:AMS1117-3.3
- added IC2: CP2102N-A01-GQFN28, CP2102N-A01-GQFN28:QFN50P500X500X80-29N-D, symbol CP2102N-A01-GQFN28:CP2102N-A01-GQFN28
- added J1: USB_B_Micro, Connector_USB:USB_Micro-B_Amphenol_10103594-0001LF_Horizontal, symbol Connector:USB_B_Micro
- added J2, J3: Conn_01x19_Male, Connector_PinHeader_2.54mm:PinHeader_1x19_P2.54mm_Vertical, symbol Connector:Conn_01x19_Male
- added Q1, Q2: SS8050-G, SS8050-G:SOT95P240X115-3N, symbol SS8050-G:SS8050-G
- added R10: 22.1K(5%), Resistor_SMD:R_0402_1005Metric, symbol Device:R
- added R11: 47.5k(5%), Resistor_SMD:R_0402_1005Metric, symbol Device:R
- added R12, R14, R9: 2k(5%), Resistor_SMD:R_0402_1005Metric, symbol Device:R
- added R13, R7: 10k(5%)(NC), Resistor_SMD:R_0402_1005Metric, symbol Device:R
- added R4, R5: 10k(5%), Resistor_SMD:R_0402_1005Metric, symbol Device:R
- added R6, R8: 0R(5%), Resistor_SMD:R_0402_1005Metric, symbol Device:R
- added SW1, SW2: SW_Push, Button_Switch_SMD:SW_SPST_B3U-1000P, symbol Switch:SW_Push
Connections:
- net GND: now also C1.2, C2.2, C3.2, C4.1, C5.2, C6.2, C7.2, C8.2, C9.1, D4.1 (K), D6.1 (K), J1.5 (GND), J1.6 (Shield), R11.1, R13.1, SW1.1, SW2.1
- net SD2: now reaches U1.17 (SHD/SD2)
- net SD3: now reaches U1.18 (SWP/SD3)
- net CMD: now reaches U1.19 (SCS/CMD)
- net CLK: now reaches U1.20 (SCK/CLK)
- net SD0: now reaches U1.21 (SDO/SD0)
- net SD1: now reaches U1.22 (SDI/SD1)
- net EN: now reaches U1.3 (EN)
- net EN: now also C6.1, C9.2, R7.1, SW2.2
- net RXD0: now reaches U1.34 (RXD0/IO3)
- net RXD0: now also R8.2
- net TXD0: now reaches U1.35 (TXD0/IO1)
- net TXD0: now also R6.2
- new net: D4.2 (A), R9.1
- new net: D6.2 (A), R14.1
- new net: R10.2, R11.2
- new net +5V: C1.1, R9.2
- new net DTR: R4.2
- new net IO0: C4.2, SW1.2
- new net RTS: R5.2
- new net RXD: R6.1
- new net TXD: R8.1
- new net USB_DN: J1.2 (D-)
- new net USB_DP: J1.3 (D+)
- new net VBUS: J1.1 (VBUS), R10.1
- new net VDD33: C2.1, C3.1, C5.1, C7.1, C8.1, R12.1, R7.2
- no-connect marks 0 -> 17
Other:
- note added: "5V->3.3V"
- note added: "Auto program DTR RTS-->EN IO0 1 1 1 1 0 0 1 1 1 0 0 1 0 1 1 0"
- note added: "Bootup"
- note added: "Bypass Capacitors"
- note added: "MicroUSB"
- note added: "USB-to-Serial"
- note added: "Voltage Regulator"
- moved on the sheet: D1, D2, D3, R1, R2, R3, U1

Commit message: FABRICATION
Parts:
- removed D3: LED, LED_SMD:LED_Cree-XHP50_3V_HighDensity, symbol Device:LED
- removed D6: LED, LED_SMD:LED_0603_1608Metric, symbol Device:LED
- removed R14: 2k(5%), Resistor_SMD:R_0402_1005Metric, symbol Device:R
- removed R2, R3: R, symbol Device:R
- renumbered D1 to led1, D2 to led2
Connections:
- net at led2.2 (A): now also R1.2, led1.2 (A)
