File: physical robot/PCB/Camera/Camera.kicad_pcb (KiCad board)
At the start: 2 copper layers, 35.8 x 47.7 mm, 60 parts, among them U1 TLV74315, U2 TLV74328, X1 CAMERA_OV2640

Commit message: pcb finiished
Parts:
- removed JP2: , 2X09-BIG
- added C14: 22uF/10V(20%), Capacitor_SMD:C_0603_1608Metric, F.Cu at (159.3, 125.1)
- added C15: 22uF/10V(20%), Capacitor_SMD:C_0603_1608Metric, F.Cu at (158.4, 132.1)
- added C16: 4.7uF/6.3V(10%), Capacitor_SMD:C_0402_1005Metric, F.Cu at (157.9, 128.9)
- added C17: 0.1uF/50V(10%)(NC), Capacitor_SMD:C_0402_1005Metric, F.Cu at (153.9, 137.6)
- added C18: 0.1uF/50V(10%), Capacitor_SMD:C_0402_1005Metric, F.Cu at (157.9, 127.8)
- added C19: 0.1uF/50V(10%), Capacitor_SMD:C_0402_1005Metric, F.Cu at (160.0, 130.0)
- added C20: 22uF/10V(20%), Capacitor_SMD:C_0603_1608Metric, F.Cu at (159.3, 121.7)
- added C21: 0.1uF/50V(10%), Capacitor_SMD:C_0402_1005Metric, F.Cu at (157.9, 130.1)
- added C22: 0.1uF/50V(10%)(NC), Capacitor_SMD:C_0402_1005Metric, F.Cu at (136.8, 136.4)
- added D2: LED, LED_SMD:LED_0603_1608Metric, F.Cu at (157.5, 125.2)
- added D3: LESD5D5.0CT1G, LESD5D5.0CT1G:LESD5D50CT1G, F.Cu at (146.3, 136.0)
- added D4: LESD5D5.0CT1G, LESD5D5.0CT1G:LESD5D50CT1G, F.Cu at (144.3, 136.1)
- added D5: LESD5D5.0CT1G, LESD5D5.0CT1G:LESD5D50CT1G, F.Cu at (142.3, 136.0)
- added D6: BAT760-7, BAT760-7:SOD2513X120N, F.Cu at (141.5, 132.8)
- added D7: LED, LED_SMD:LED_0603_1608Metric, F.Cu at (151.0, 124.9)
- added G***: LOGO, LOGO, F.Cu at (140.0, 86.9)
- added G***: LOGO, LOGO, B.Cu at (140.9, 87.0)
- added IC1: AMS1117-3.3, AMS1117-3.3:SOT229P700X180-4N, F.Cu at (148.5, 128.5)
- added IC2: CP2102N-A01-GQFN28, CP2102N-A01-GQFN28:QFN50P500X500X80-29N-D, F.Cu at (140.2, 123.3)
- added J1: USB_B_Micro, Connector_USB:USB_Micro-B_Amphenol_10103594-0001LF_Horizontal, F.Cu at (147.7, 143.7)
- added Q1: SS8050-G, SS8050-G:SOT95P240X115-3N, F.Cu at (158.2, 138.1)
- added Q2: SS8050-G, SS8050-G:SOT95P240X115-3N, F.Cu at (151.4, 136.7)
- added R10: 10k(5%), Resistor_SMD:R_0402_1005Metric, F.Cu at (158.2, 143.5)
- added R11: 22.1K(5%), Resistor_SMD:R_0402_1005Metric, F.Cu at (138.1, 129.9)
- added R12: 10k(5%)(NC), Resistor_SMD:R_0402_1005Metric, F.Cu at (160.4, 132.4)
- added R13: 47.5k(5%), Resistor_SMD:R_0402_1005Metric, F.Cu at (138.1, 128.8)
- added R14: 2k(5%), Resistor_SMD:R_0402_1005Metric, F.Cu at (138.1, 131.2)
- added R15: 10k(5%)(NC), Resistor_SMD:R_0402_1005Metric, F.Cu at (138.1, 132.6)
- added R16: 2k(5%), Resistor_SMD:R_0402_1005Metric, F.Cu at (147.1, 123.5)
- added R3: 2k(5%), Resistor_SMD:R_0402_1005Metric, F.Cu at (157.7, 121.5)
- added R7: 0R(5%), Resistor_SMD:R_0402_1005Metric, F.Cu at (147.9, 136.0)
- added R8: 0R(5%), Resistor_SMD:R_0402_1005Metric, F.Cu at (149.0, 136.0)
- added R9: 10k(5%), Resistor_SMD:R_0402_1005Metric, F.Cu at (148.6, 123.6)
- added REF**: OSHW-Logo2_14.6x12mm_SilkScreen, Symbol:OSHW-Logo2_14.6x12mm_SilkScreen, F.Cu at (158.9, 92.4)
- added REF**: OSHW-Logo2_14.6x12mm_SilkScreen, Symbol:OSHW-Logo2_14.6x12mm_SilkScreen, B.Cu at (157.1, 94.5)
- added REF**: WEEE-Logo_14x20mm_SilkScreen, Symbol:WEEE-Logo_14x20mm_SilkScreen, B.Cu at (148.5, 109.7)
- added SW1: SW_Push, Button_Switch_SMD:SW_SPST_B3U-1000P, F.Cu at (154.0, 131.1)
- added SW2: SW_Push, Button_Switch_SMD:SW_SPST_B3U-1000P, F.Cu at (139.2, 137.1)
- added U3: ESP32-WROOM-32, RF_Module:ESP32-WROOM-32, B.Cu at (145.8, 130.3)
- U2: value TLV74328 -> OV5640
Connections:
- U2 pad 1: 3.3V -> GND
- U2 pad 2: GND -> Net-(U1-VDD)
- U2 pad 3: 3.3V -> Net-(U1-IO26)
- U2 pad 4: (no net) -> Net-(U1-IO27)
- U2 pad 5: 2.8V -> Net-(U1-IO23)
Routing:
- net GND: track 123.3 -> 265.8 mm, vias 35 -> 53
- net /VDD33: track 0.00 -> 81.7 mm, vias 0 -> 10
- net /EN: track 0.00 -> 71.2 mm, vias 0 -> 3
- net +5V: track 0.00 -> 62.8 mm, vias 0 -> 2
- net /IO4: track 0.00 -> 43.8 mm, vias 0 -> 2
- net /IO21: track 0.00 -> 40.6 mm, vias 0 -> 2
- net /USB_DP: track 0.00 -> 40.5 mm, vias 0 -> 2
- net /IO18: track 0.00 -> 40.2 mm, vias 0 -> 4
- net /IO5: track 0.00 -> 39.3 mm, vias 0 -> 4
- net /USB_DN: track 0.00 -> 38.5 mm, vias 0 -> 4
- net /IO23: track 0.00 -> 34.8 mm, vias 0 -> 1
- net /VBUS: track 0.00 -> 32.7 mm, vias 0 -> 1
- net /IO22: track 0.00 -> 31.2 mm, vias 0 -> 2
- net /RTS: track 0.00 -> 30.5 mm, vias 0 -> 2
- net Net-(Q1-Pad1): track 0.00 -> 23.3 mm
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Other:
- board size 35.8 x 47.7 mm -> 35.8 x 71.3 mm
- board text added: "Designed by Dexter R. Shepherd"
- board text added: "Embedded Computer vision Module (ECVM)"

Commit message: FABRICATION
Parts:
- added R1: R_0603_1608Metric, Resistor_SMD:R_0603_1608Metric, F.Cu at (164.4, 88.7)
- added led1: LED_D5.0mm_Horizontal_O6.35mm_Z15.0mm, LED_THT:LED_D5.0mm_Horizontal_O6.35mm_Z15.0mm, F.Cu at (161.5, 83.6)
- added led2: LED_D5.0mm_Horizontal_O6.35mm_Z15.0mm, LED_THT:LED_D5.0mm_Horizontal_O6.35mm_Z15.0mm, F.Cu at (133.8, 86.0)
- C1, C7: value 0.1uF -> 22uF/10V(20%)
- C2: value 10uF -> 22uF/10V(20%)
- C3: value 10uF -> 4.7uF/6.3V(10%)
- C4: value 0.1uF -> 0.1uF/50V(10%)(NC)
- C5: value 0.1uF -> 0.1uF/50V(10%)
- C6: value 22pF -> 0.1uF/50V(10%)
- C8: value 1.0uF -> 0.1uF/50V(10%)
- C9: value 10uF -> 0.1uF/50V(10%)(NC)
- D1: value GREEN -> LED
- D2: value LED -> (none)
- D3: value LESD5D5.0CT1G -> LED
- D6: value BAT760-7 -> LED
- R1, R2: value 10K -> R
- R10: value 10k(5%) -> 22.1K(5%)
- R11: value 22.1K(5%) -> 47.5k(5%)
- R12: value 10k(5%)(NC) -> 2k(5%)
- R13: value 47.5k(5%) -> 10k(5%)(NC)
- R3: value 2k(5%) -> R
- R4, R5: value 10K -> 10k(5%)
- R6: value 10K -> 0R(5%)
- R7: value 0R(5%) -> 10k(5%)(NC)
- R9: value 10k(5%) -> 2k(5%)
- U1: value TLV74315 -> ESP32-WROOM-32
Connections:
- C1 pad 1: 3.3V -> +5V
- C2 pad 1: 3.3V -> /VDD33
- C3 pad 1: 2.8V -> /VDD33
- C4 pad 1: ~{RESET} -> GND
- C4 pad 2: GND -> /IO0
- C5 pad 1: 2.8V -> /VDD33
- C6 pad 1: PCLK -> /EN
- C7 pad 1: 1.5V -> /VDD33
- C8 pad 1: 1.5V -> /VDD33
- C9 pad 1: 2.8V -> GND
- C9 pad 2: GND -> /EN
- D1 pad A: N$3 -> (no net)
- D1 pad C: GND -> (no net)
- D3 pad 1: /USB_DN -> GND
- D3 pad 2: GND -> Net-(D3-A)
- D6 pad 1: +5V -> GND
- D6 pad 2: /VBUS -> Net-(D6-A)
- J1 pad 4: Net-(J1-Pad4) -> unconnected-(J1-ID-Pad4)
- R1 pad 1: 3.3V -> Net-(U1-IO17)
- R1 pad 2: N$1 -> Net-(D1-A)
- R10 pad 1: Net-(Q2-Pad1) -> /VBUS
- R10 pad 2: /RTS -> Net-(R10-Pad2)
- R11 pad 1: /VBUS -> GND
- R11 pad 2: Net-(IC2-Pad8) -> Net-(R10-Pad2)
- R12 pad 1: /EN -> /VDD33
- R12 pad 2: /VDD33 -> unconnected-(R12-Pad2)
- R13 pad 2: Net-(IC2-Pad8) -> unconnected-(R13-Pad2)
- R14 pad 1: /VDD33 -> Net-(D6-A)
- R14 pad 2: Net-(IC2-Pad9) -> unconnected-(R14-Pad2)
- R2 pad 1: 3.3V -> Net-(U1-IO32)
- R2 pad 2: SCL -> Net-(D2-A)
- R3 pad 1: Net-(D1-Pad2) -> Net-(U1-IO33)
- R3 pad 2: +5V -> Net-(D3-A)
- R4 pad 1: 3.3V -> unconnected-(R4-Pad1)
- R4 pad 2: SDA -> /DTR
- R5 pad 1: 3.3V -> unconnected-(R5-Pad1)
- R5 pad 2: ~{RESET} -> /RTS
- R6 pad 1: PWDN -> /RXD
- R6 pad 2: GND -> /TXD0
- R7 pad 1: /RXD -> /EN
- R7 pad 2: /TXD0 -> /VDD33
- R9 pad 1: Net-(Q1-Pad1) -> Net-(D4-A)
- R9 pad 2: /DTR -> +5V
- U1 pad 1: 3.3V -> GND
- U1 pad 2: GND -> Net-(U1-VDD)
- U1 pad 3: 3.3V -> /EN
- U1 pad 4: (no net) -> Net-(U1-SENSOR_VP)
- U1 pad 5: 1.5V -> Net-(U1-SENSOR_VN)
Routing:
- net /IO17: track 0.00 -> 109.9 mm, vias 0 -> 9
- net GND: track 265.8 -> 277.3 mm, vias 53 -> 55
- net (no net): track 28.8 -> 37.1 mm
- net ~{RESET}: track 49.4 -> 50.2 mm, vias 2 -> 0
- net /VDD33: track 81.7 -> 81.0 mm
- net 1.5V: track 95.6 -> 95.9 mm, vias 5 -> 0
- net SDA: vias 1 -> 0
- net SCL: vias 3 -> 0
- net PCLK: vias 7 -> 0
- net Net-(U1-SENSOR_VN): vias 0 -> 5
- net Net-(D2-A): vias 0 -> 3
- net 2.8V: vias 2 -> 0
- net /RTS: vias 2 -> 4
- net /EN: vias 3 -> 10
- net /DTR: vias 0 -> 1

Commit message: Update Camera.kicad_pcb
Other:
- board size 35.8 x 71.3 mm -> 36.2 x 71.7 mm
